File: interfaces.kicad_sch (KiCad schematic)
At the start: 6 parts, among them P2 SMA Jack, Female, P3 Conn_01x04_Male, U3 SX1276IMLTRT

Commit message: Add partial RF and Memory wiring and placement
Parts:
- removed P2: SMA Jack, Female, KKicadLib:SMA_Female_Edge_60312202114513, symbol KKicadLib:SMA Jack, Female
- removed U3: SX1276IMLTRT, QFN65P600X600X100-29N, symbol kkicadlib:SX1276IMLTRT
- added DB1, DB2, DB3: TestPoint, TestPoint:TestPoint_Pad_1.5x1.5mm, symbol Connector:TestPoint
Other:
- title: (none) -> LoRa Expansion Card for Frame.Work Laptop
Changed lines of the file:
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@@
 (kicad_sch (version 20211123) (generator eeschema)
   (paper "A4")
+  (title_block
+    (title "LoRa Expansion Card for Frame.Work Laptop")
+    (rev "0.1.0")
+    (comment 3 "Kris Keillor")
+  )
+  (symbol (lib_id "Connector:TestPoint") (at 207.01 137.16 0) (unit 1)
+    (in_bom yes) (on_board yes)
+    (property "Reference" "DB3" (id 0) (at 208.4832 134.1628 0)
+      (effects (font (size 1.27 1.27)) (justify left))
+    )
+    (property "Value" "TestPoint" (id 1) (at 208.4832 136.4742 0)
+      (effects (font (size 1.27 1.27)) (justify left))
+    )
+    (property "Footprint" "TestPoint:TestPoint_Pad_1.5x1.5mm" (id 2) (at 212.09 137.16 0)
+      (effects (font (size 1.27 1.27)) hide)
+    )
+    (property "Datasheet" "~" (id 3) (at 212.09 137.16 0)
+      (effects (font (size 1.27 1.27)) hide)
+    )
+    (pin "1")
+  )
   (symbol (lib_id "Device:LED") (at 186.69 83.82 180) (unit 1)
     (in_bom yes) (on_board yes) (fields_autoplaced)
@@
     (pin "2")
   )
-  (symbol (lib_id "kkicadlib:SX1276IMLTRT") (at 109.22 87.63 0) (unit 1)
-    (in_bom yes) (on_board yes) (fields_autoplaced)
-    (property "Reference" "U3" (id 0) (at 109.22 49.53 0))
-    (property "Value" "SX1276IMLTRT" (id 1) (at 109.22 52.07 0))
-    (property "Footprint" "QFN65P600X600X100-29N" (id 2) (at 109.22 87.63 0)
-      (effects (font (size 1.27 1.27)) (justify bottom) hide)
+  (symbol (lib_id "Connector:TestPoint") (at 195.58 137.16 0) (unit 1)
+    (in_bom yes) (on_board yes)
+    (property "Reference" "DB2" (id 0) (at 197.0532 134.1628 0)
+      (effects (font (size 1.27 1.27)) (justify left))
     )
-    (property "Datasheet" "" (id 3) (at 109.22 87.63 0)
+    (property "Value" "TestPoint" (id 1) (at 197.0532 136.4742 0)
+      (effects (font (size 1.27 1.27)) (justify left))
+    )
+    (property "Footprint" "TestPoint:TestPoint_Pad_1.5x1.5mm" (id 2) (at 200.66 137.16 0)
       (effects (font (size 1.27 1.27)) hide)
     )
-    (property "STANDARD" "IPC-7351B" (id 4) (at 109.22 87.63 0)
-      (effects (font (size 1.27 1.27)) (justify bottom) hide)
-    )
-    (property "MANUFACTURER" "Semtech Corporation" (id 5) (at 109.22 87.63 0)
-      (effects (font (size 1.27 1.27)) (justify bottom) hide)
-    )
-    (property "PARTREV" "5" (id 6) (at 109.22 87.63 0)
-      (effects (font (size 1.27 1.27)) (justify bottom) hide)
+    (property "Datasheet" "~" (id 3) (at 200.66 137.16 0)
+      (effects (font (size 1.27 1.27)) hide)
     )
     (pin "1")
-    (pin "10")
-    (pin "11")
-    (pin "12")
-    (pin "13")
-    (pin "14")
-    (pin "15")
-    (pin "16")
-    (pin "17")
-    (pin "18")
-    (pin "19")
-    (pin "2")
-    (pin "20")
-    (pin "21")
-    (pin "22")
-    (pin "23")
-    (pin "24")
-    (pin "25")
-    (pin "26")
-    (pin "27")
-    (pin "28")
-    (pin "29")
-    (pin "3")
-    (pin "4")
-    (pin "5")
-    (pin "6")
-    (pin "7")
-    (pin "8")
-    (pin "9")
-  )
-  (symbol (lib_id "KKicadLib:SMA Jack, Female") (at 181.61 38.1 0) (unit 1)
-    (in_bom yes) (on_board yes) (fields_autoplaced)
-    (property "Reference" "P2" (id 0) (at 182.8935 30.48 0))
-    (property "Value" "SMA Jack, Female" (id 1) (at 182.8935 33.02 0))
-    (property "Footprint" "KKicadLib:SMA_Female_Edge_60312202114513" (id 2) (at 181.61 38.1 0)
-      (effects (font (size 1.27 1.27)) (justify bottom) hide)
-    )
-    (property "Datasheet" "" (id 3) (at 181.61 38.1 0)
-      (effects (font (size 1.27 1.27)) hide)
-    )
-    (property "DATASHEET-URL" "https://www.we-online.com/catalog/datasheet/60312202114513.pdf" (id 4) (at 181.61 38.1 0)
-      (effects (font (size 1.27 1.27)) (justify bottom) hide)
-    )
-    (property "INTERFACE" "MIL-STD-348" (id 5) (at 181.61 38.1 0)
-      (effects (font (size 1.27 1.27)) (justify bottom) hide)
-    )
-    (property "VALUE" "60312202114513" (id 6) (at 181.61 38.1 0)
-      (effects (font (size 1.27 1.27)) (justify bottom) hide)
-    )
-    (property "ORIENTATION-TYPE" "Straight" (id 7) (at 181.61 38.1 0)
-      (effects (font (size 1.27 1.27)) (justify bottom) hide)
-    )
-    (property "MOUNT" "End Launch" (id 8) (at 181.61 38.1 0)
-      (effects (font (size 1.27 1.27)) (justify bottom) hide)
-    )
-    (property "PART-NUMBER" "60312202114513" (id 9) (at 181.61 38.1 0)
-      (effects (font (size 1.27 1.27)) (justify bottom) hide)
-    )
-    (property "Z" "50Ohm" (id 10) (at 181.61 38.1 0)
-      (effects (font (size 1.27 1.27)) (justify bottom) hide)
-    )
-    (property "GENDER" "Jack" (id 11) (at 181.61 38.1 0)
-      (effects (font (size 1.27 1.27)) (justify bottom) hide)
-    )
-    (pin "1")
-    (pin "2")
-    (pin "3")
-    (pin "4")
-    (pin "5")
   )
   (symbol (lib_id "Device:LED") (at 186.69 106.68 180) (unit 1)
@@
     (pin "2")
   )
+  (symbol (lib_id "Connector:TestPoint") (at 184.15 137.16 0) (unit 1)
+    (in_bom yes) (on_board yes)
+    (property "Reference" "DB1" (id 0) (at 185.6232 134.1628 0)
+      (effects (font (size 1.27 1.27)) (justify left))
+    )
+    (property "Value" "TestPoint" (id 1) (at 185.6232 136.4742 0)
+      (effects (font (size 1.27 1.27)) (justify left))
+    )
+    (property "Footprint" "TestPoint:TestPoint_Pad_1.5x1.5mm" (id 2) (at 189.23 137.16 0)
+      (effects (font (size 1.27 1.27)) hide)
+    )
+    (property "Datasheet" "~" (id 3) (at 189.23 137.16 0)
+      (effects (font (size 1.27 1.27)) hide)
+    )
+    (pin "1")
+  )
   (symbol (lib_id "Connector:Conn_01x04_Male") (at 184.15 60.96 0) (unit 1)
